Commit message: fix(ot/sim): resolve Gazebo joint mismatch and integrate BehaviorTree.CPP v4 motor publisher
- Sync amr.urdf joint names with libgazebo_ros_diff_drive. so configuration to prevent hardware paralysis
- Implement geometry_msgs/Twist publisher inside MoveToStation action node to drive robot wheels at 20Hz
- Enable full X11 display session pass-through to popup Gazebo 3D GUI smoothly on Ubuntu desktop

File: ros2_ws/src/smart_factory_sim/urdf/amr.urdf (robot description, URDF)
Before this commit: robot smart_amr, 2 links, 1 joints
Links:
- added link left_wheel, mass 2.0; collision cylinder length=0.05 radius=0.1; visual cylinder length=0.05 radius=0.1
- added link right_wheel, mass 2.0; collision cylinder length=0.05 radius=0.1; visual cylinder length=0.05 radius=0.1
- link base_link: mass 20.0 -> 15.0
- link laser_link: mass None -> 0.1; geometry visual cylinder length=0.06 radius=0.05
Joints:
- removed joint laser_joint
- added joint laser_link_joint: type fixed, parent base_link, child laser_link, origin xyz=0.2 0 0.13 rpy=0 0 0
- added joint left_wheel_joint: type continuous, parent base_link, child left_wheel, origin xyz=-0.15 0.225 -0.05 rpy=-1.5708 0 0, axis 0 0 1
- added joint right_wheel_joint: type continuous, parent base_link, child right_wheel, origin xyz=-0.15 -0.225 -0.05 rpy=-1.5708 0 0, axis 0 0 1

Commit message: fix(twin/media): resolve camera occlusion and enhance lidar fault detection logic
- Adjust camera <near> clipping plane to 0.12 to pass through robot bounding box
- Fix false-positive brake triggers by checking full laser scan array for infinity values
- Integrate Gazebo /amr_front_camera/image_raw topic into GStreamer appsrc pipeline
- Map WebRTC remote description answer and ICE candidates directly to webrtcbin
- Build factory_zone.world infrastructure with boxes and walls to provide valid lidar ranges

File: ros2_ws/src/smart_factory_sim/urdf/amr.urdf (robot description, URDF)
Before this commit: robot amr_01, 4 links, 3 joints
Links:
- added link camera_link; visual box size=0.05 0.05 0.05
Joints:
- added joint camera_joint: type fixed, parent base_link, child camera_link, origin xyz=0.4 0.0 0.25 rpy=0 0 0
